Commit message: revised urdf files

File: robots/hsrb4s_with_fake_joints.urdf.xacro (robot description, xacro)
@@ -25,52 +25,31 @@
 POSSIBILITY OF SUCH DAMAGE.
 -->
-<robot name="hsrb"
-       xmlns:controller="http://playerstage.sourceforge.net/gazebo/xmlschema/#controller"
-       xmlns:interface="http://playerstage.sourceforge.net/gazebo/xmlschema/#interface"
-       xmlns:sensor="http://playerstage.sourceforge.net/gazebo/xmlschema/#sensor"
-       xmlns:xacro="http://ros.org/wiki/xacro">
-    <!-- common xacro -->
-    <xacro:include filename="$(find hsr_description)/urdf/common.xacro" />
-    <xacro:include filename="$(find hsr_description)/urdf/materials.urdf.xacro" />
-    <!-- links and joints -->
-    <xacro:include filename="$(find hsr_description)/urdf/base_v2_with_fake_joints/base.urdf.xacro" />
-    <xacro:include filename="$(find hsr_description)/urdf/torso_v0/torso.urdf.xacro" />
-    <xacro:include filename="$(find hsr_description)/urdf/head_v2/head.urdf.xacro" />
-    <xacro:include filename="$(find hsr_description)/urdf/arm_v0/arm.urdf.xacro" />
-    <xacro:include filename="$(find hsr_description)/urdf/wrist_v0/wrist.urdf.xacro" />
-    <xacro:include filename="$(find hsr_description)/urdf/hand_v0/hand.urdf.xacro" />
-    <!-- This switches a format of mesh files for visual property -->
-    <xacro:arg name="use_obj_for_visual" default="false" />
-    <xacro:property name="g_use_obj_for_visual" value="$(arg use_obj_for_visual)"/>
-    <!-- constant -->
-    <xacro:property name="g_robot_name" value="hsrb"/>
-    <!-- create robot -->
-    <xacro:hsrb_base prefix="base" robot_namespace="${g_robot_name}"/>
-    <xacro:hsrb_torso prefix="torso" parent="base_link" mimic_joint="arm_lift_joint">
-        <origin xyz="0.0 0.0 0.752" rpy="0.0 0.0 0.0"/>
-    </xacro:hsrb_torso>
-    <xacro:hsrb_head prefix="head" parent="torso_lift_link">
-        <origin xyz="0.0 0.0 0.0" rpy="0.0 0.0 0.0"/>
-    </xacro:hsrb_head>
-    <xacro:hsrb_arm prefix="arm" parent="base_link">
-        <origin xyz="0.0 0.0 0.340" rpy="0.0 0.0 0.0"/>
-    </xacro:hsrb_arm>
-    <xacro:hsrb_wrist prefix="wrist" parent="arm_roll_link" robot_namespace="${g_robot_name}">
-        <origin xyz="0.0 0.0 0.0" rpy="0.0 0.0 0.0"/>
-    </xacro:hsrb_wrist>
-    <xacro:hsrb_hand prefix="hand" parent="wrist_roll_link">
-        <origin xyz="0.012 0.0 0.1405" rpy="0.0 0.0 ${pi}"/>
-    </xacro:hsrb_hand>
-    <gazebo>
-        <plugin name="${g_robot_name}_ros_control" filename="lib${g_robot_name}_gazebo_ros_control.so">
-            <robotNamespace>${g_robot_name}</robotNamespace>
-        </plugin>
-        <plugin name="${g_robot_name}_p3d_ground_truth" filename="libgazebo_ros_p3d.so">
-            <robotNamespace>${g_robot_name}</robotNamespace>
-            <bodyName>base_footprint</bodyName>
-            <topicName>odom_ground_truth</topicName>
-            <frameName>map</frameName>
-            <updateRate>30</updateRate>
-        </plugin>
-    </gazebo>
+<robot name="hsrb">
+    <include filename="$(find hsr_description)/robots/hsrb4s.urdf.xacro" />
+    <link name="odom"/>
+    <joint name="odom_x" type="prismatic">
+        <axis xyz="1.0 0.0 0.0" />
+        <limit effort="1.0" velocity="0.1" lower="-10.0" upper="10.0" />
+        <parent link="odom" />
+        <child link="odom_x_link" />
+    </joint>
+     <link name="odom_x_link"/>
+    <joint name="odom_y" type="prismatic">
+        <axis xyz="0.0 1.0 0.0" />
+        <limit effort="1.0" velocity="0.1" lower="-10.0" upper="10.0" />
+        <parent link="odom_x_link" />
+        <child link="odom_y_link" />
+    </joint>
+     <link name="odom_y_link"/>
+    <joint name="odom_t" type="continuous">
+        <axis xyz="0.0 0.0 1.0" />
+        <limit effort="1.0" velocity="0.1"/>
+        <parent link="odom_y_link" />
+        <child link="odom_t_link" />
+    </joint>
+    <link name="odom_t_link"/>
+    <joint name="hsrb" type="fixed">
+        <parent link="odom_t_link" />
+        <child link="base_footprint" />
+    </joint>
 </robot>
