Commit message: adjusted joint limits

File: urdf/arm_v0/arm.urdf.xacro (robot description, xacro)
@@ -33,5 +33,7 @@
             <xacro:insert_block name="origin" />
             <axis xyz="0.0 0.0 1.0" />
-            <limit effort="100.0" velocity="0.2" lower="0.0" upper="0.69" />
+            <!--limit effort="100.0" velocity="0.2" lower="0.0" upper="0.69" /-->
+            <limit effort="100.0" velocity="0.2" lower="0.005" upper="0.67" />
+	    	<safety_controller k_position="100" k_velocity="200000" soft_lower_limit="0.005" soft_upper_limit="0.67"/>
             <parent link="${parent}" />
             <child link="${prefix}_lift_link" />
@@ -64,5 +66,7 @@
             <origin xyz="0.141 0.078 0.0" rpy="0.0 0.0 0.0" />
             <axis xyz="0.0 -1.0 0.0" />
-            <limit effort="100.0" velocity="1.2" lower="-2.62" upper="0.0" />
+            <!--limit effort="100.0" velocity="1.2" lower="-2.62" upper="0.0" /-->
+            <limit effort="100.0" velocity="1.2" lower="-2.61" upper="-0.02" />
+	    	<safety_controller k_position="100" k_velocity="200000" soft_lower_limit="-2.61" soft_upper_limit="-0.02"/>
             <parent link="${prefix}_lift_link" />
             <child link="${prefix}_flex_link" />
@@ -95,5 +99,7 @@
             <origin xyz="0.005 0.0 0.345" rpy="0.0 0.0 0.0" />
             <axis xyz="0.0 0.0 1.0" />
-            <limit effort="100.0" velocity="2.0" lower="-2.09" upper="3.84" />
+            <!--limit effort="100.0" velocity="2.0" lower="-2.09" upper="3.84" /-->
+            <limit effort="100.0" velocity="2.0" lower="-1.95" upper="3.67" />
+	    	<safety_controller k_position="100" k_velocity="200000" soft_lower_limit="-1.95" soft_upper_limit="3.67"/>
             <parent link="${prefix}_flex_link" />
             <child link="${prefix}_roll_link" />

File: urdf/head_v2/head.urdf.xacro (robot description, xacro)
@@ -36,5 +36,7 @@
             <xacro:insert_block name="origin" />
             <axis xyz="0.0 0.0 1.0" />
-            <limit effort="100.0" velocity="1.0" lower="-3.84" upper="1.75" />
+            <!--limit effort="100.0" velocity="1.0" lower="-3.84" upper="1.75" /-->
+            <limit effort="100.0" velocity="1.0" lower="-3.83" upper="1.74" />
+            <safety_controller k_position="100" k_velocity="200000" soft_lower_limit="-3.83" soft_upper_limit="1.74"/>
             <parent link="${parent}" />
             <child link="${prefix}_pan_link" />
@@ -67,5 +69,7 @@
             <origin xyz="0.02 0.0 0.0" rpy="0.0 0.0 0.0" />
             <axis xyz="0.0 -1.0 0.0" />
-            <limit effort="100.0" velocity="1.0" lower="-1.57" upper="0.52" />
+            <!--limit effort="100.0" velocity="1.0" lower="-1.57" upper="0.52" /-->
+            <limit effort="100.0" velocity="1.0" lower="-1.56" upper="0.47" />
+            <safety_controller k_position="100" k_velocity="200000" soft_lower_limit="-1.56" soft_upper_limit="0.47"/>
             <parent link="${prefix}_pan_link" />
             <child link="${prefix}_tilt_link" />

File: urdf/wrist_v0/wrist.urdf.xacro (robot description, xacro)
@@ -34,5 +34,7 @@
             <origin xyz="0.0 0.0 0.0" rpy="0.0 0.0 0.0" />
             <axis xyz="0.0 -1.0 0.0" />
-            <limit effort="100.0" velocity="1.5" lower="-1.92" upper="1.22" />
+            <!--limit effort="100.0" velocity="1.5" lower="-1.92" upper="1.22" /-->
+            <limit effort="100.0" velocity="1.5" lower="-1.91" upper="1.21" />
+            <safety_controller k_position="100" k_velocity="200000" soft_lower_limit="-1.91" soft_upper_limit="1.21"/>
             <parent link="${parent}" />
             <child link="${prefix}_flex_link" />
@@ -74,5 +76,7 @@
             <origin xyz="0.0 0.0 0.0" rpy="0.0 0.0 0.0" />
             <axis xyz="0.0 0.0 1.0" />
-            <limit effort="100.0" velocity="1.5" lower="-1.92" upper="3.67" />
+            <!--limit effort="100.0" velocity="1.5" lower="-1.92" upper="3.67" /-->
+            <limit effort="100.0" velocity="1.5" lower="-1.91" upper="3.63" />
+            <safety_controller k_position="100" k_velocity="200000" soft_lower_limit="-1.91" soft_upper_limit="3.63"/>
             <parent link="${prefix}_flex_link" />
             <child link="${prefix}_roll_link" />

Commit message: fixed arm lift joint limits

File: urdf/arm_v0/arm.urdf.xacro (robot description, xacro)
@@ -34,5 +34,5 @@
             <axis xyz="0.0 0.0 1.0" />
             <!--limit effort="100.0" velocity="0.2" lower="0.0" upper="0.69" /-->
-            <limit effort="100.0" velocity="0.2" lower="0.005" upper="0.67" />
+            <limit effort="100.0" velocity="0.15" lower="0.005" upper="0.67" />
 	    	<safety_controller k_position="100" k_velocity="200000" soft_lower_limit="0.005" soft_upper_limit="0.67"/>
             <parent link="${parent}" />
@@ -67,6 +67,6 @@
             <axis xyz="0.0 -1.0 0.0" />
             <!--limit effort="100.0" velocity="1.2" lower="-2.62" upper="0.0" /-->
-            <limit effort="100.0" velocity="1.2" lower="-2.61" upper="-0.02" />
-	    	<safety_controller k_position="100" k_velocity="200000" soft_lower_limit="-2.61" soft_upper_limit="-0.02"/>
+            <limit effort="100.0" velocity="1.2" lower="-2.61" upper="-0.03" />
+	    	<safety_controller k_position="100" k_velocity="200000" soft_lower_limit="-2.61" soft_upper_limit="-0.03"/>
             <parent link="${prefix}_lift_link" />
             <child link="${prefix}_flex_link" />

File: urdf/torso_v0/torso.urdf.xacro (robot description, xacro)
@@ -33,5 +33,5 @@
             <!-- <origin xyz="0.0 0.0 0.752" rpy="0.0 0.0 0.0" /> -->
             <axis xyz="0.0 0.0 1.0" />
-            <limit effort="100.0" velocity="0.1" lower="0.0" upper="0.345" />
+            <limit effort="100.0" velocity="0.075" lower="0.0025" upper="0.335" />
             <parent link="${parent}" />
             <child link="${prefix}_lift_link" />

Commit message: commented out inertia entries rviz is complaining about

File: urdf/arm_v0/arm.urdf.xacro (robot description, xacro)
@@ -42,10 +42,10 @@
         </joint>
         <link name="${prefix}_flex_link">
-            <inertial>
+<!--             <inertial>
                 <mass value="1.339295"/>
                 <origin xyz="0.000632 0.006404 0.118529"/>
                 <inertia ixx="7.528" ixy="-0.000020284207" ixz="-0.000022947194"
                     iyy="0.007102" iyz="-0.000091796075" izz="0.001552"/>
-            </inertial>
+            </inertial> -->
             <visual>
                 <geometry>

File: urdf/base_v2/base.urdf.xacro (robot description, xacro)
@@ -112,5 +112,5 @@
         </joint>
         <link name="${prefix}_${suffix}_bumper_link">
-            <inertial>
+<!--             <inertial>
                 <origin xyz="0.0 0.0 0.0" />
                 <mass value="0.06"/>
@@ -118,5 +118,5 @@
                     ixx="0.001437"  ixy="0.0"  ixz="0.0"
                     iyy="0.001437" iyz="0.0" izz="0.002875" />
-            </inertial>
+            </inertial> -->
             <visual>
                 <geometry>

File: urdf/hand_v0/hand.urdf.xacro (robot description, xacro)
@@ -170,5 +170,5 @@
         </xacro:hsrb_finger_distal_base>
         <link name="${prefix}_${suffix}_distal_link">
-            <inertial>
+<!--             <inertial>
                 <mass value="0.027731"/>
                 <origin xyz="0.011116 0.005679 0.017532"/>
@@ -176,5 +176,5 @@
                     ixx="0.000004451952" ixy="-0.000000617574" ixz="0.000000503765"
                     iyy="0.000000503765" iyz="-0.000000435048" izz="0.000004456764"/>
-            </inertial>
+            </inertial> -->
             <visual>
                 <geometry>
