Commit message: added bumpers and made ft sensor revolute like the hsr description on the robot

File: urdf/base_v2/base.urdf.xacro (robot description, xacro)
@@ -178,4 +178,50 @@
             </collision>
         </link>
+        <joint name="${prefix}_f_bumper_joint" type="revolute">
+            <origin rpy="0.0 0.0 0.0" xyz="0.0 0.0 0.0"/>
+            <parent link="${prefix}_link"/>
+            <child link="${prefix}_f_bumper_link"/>
+            <limit effort="0" lower="0" upper="0" velocity="0"/>
+        </joint>
+        <link name="${prefix}_f_bumper_link">
+            <inertial>
+                <origin xyz="0.0 0.0 0.0"/>
+                <mass value="0.06"/>
+                <inertia ixx="0.001437" ixy="0.0" ixz="0.0" iyy="0.001437" iyz="0.0" izz="0.002875"/>
+            </inertial>
+            <visual>
+                <geometry>
+                    <mesh filename="package://hsrb_description/meshes/base_v2/bumper.dae"/>
+                </geometry>
+            </visual>
+            <collision>
+                <geometry>
+                    <mesh filename="package://hsrb_description/meshes/base_v2/bumper.stl"/>
+                </geometry>
+            </collision>
+        </link>
+        <joint name="${prefix}_b_bumper_joint" type="revolute">
+            <origin rpy="0.0 0.0 3.141592653589793" xyz="0.0 0.0013 0.0"/>
+            <parent link="${prefix}_link"/>
+            <child link="${prefix}_b_bumper_link"/>
+            <limit effort="0" lower="0" upper="0" velocity="0"/>
+        </joint>
+        <link name="${prefix}_b_bumper_link">
+            <inertial>
+                <origin xyz="0.0 0.0 0.0"/>
+                <mass value="0.06"/>
+                <inertia ixx="0.001437" ixy="0.0" ixz="0.0" iyy="0.001437" iyz="0.0" izz="0.002875"/>
+            </inertial>
+            <visual>
+                <geometry>
+                    <mesh filename="package://hsrb_description/meshes/base_v2/bumper.dae"/>
+                </geometry>
+            </visual>
+            <collision>
+                <geometry>
+                    <mesh filename="package://hsrb_description/meshes/base_v2/bumper.stl"/>
+                </geometry>
+            </collision>
+        </link>
         <joint name="${prefix}_roll_joint" type="continuous">
             <origin xyz="0.0 0.0 0.0" rpy="0.0 0.0 0.0" />

File: urdf/sensors/ft_sensor.urdf.xacro (robot description, xacro)
@@ -28,8 +28,9 @@
     <xacro:include filename="$(find hsr_description)/urdf/sensors/ft_sensor.gazebo.xacro"/>
     <xacro:macro name="ft_sensor" params="prefix robot_namespace parent joint_name *origin">
-        <joint name="${prefix}_ft_sensor_frame_joint" type="fixed">
+        <joint name="${prefix}_ft_sensor_frame_joint" type="revolute">
             <xacro:insert_block name="origin"/>
             <parent link="${parent}"/>
             <child link="${prefix}_ft_sensor_frame"/>
+            <limit effort="100.0" lower="0" upper="0" velocity="1.5"/>
         </joint>
         <link name="${prefix}_ft_sensor_frame"/>

Commit message: commented out visuals for bumper, because they are not available in hsr_meshes

File: urdf/base_v2/base.urdf.xacro (robot description, xacro)
@@ -190,5 +190,5 @@
                 <inertia ixx="0.001437" ixy="0.0" ixz="0.0" iyy="0.001437" iyz="0.0" izz="0.002875"/>
             </inertial>
-            <visual>
+<!--             <visual>
                 <geometry>
                     <mesh filename="package://hsrb_description/meshes/base_v2/bumper.dae"/>
@@ -199,5 +199,5 @@
                     <mesh filename="package://hsrb_description/meshes/base_v2/bumper.stl"/>
                 </geometry>
-            </collision>
+            </collision> -->
         </link>
         <joint name="${prefix}_b_bumper_joint" type="revolute">
@@ -213,5 +213,5 @@
                 <inertia ixx="0.001437" ixy="0.0" ixz="0.0" iyy="0.001437" iyz="0.0" izz="0.002875"/>
             </inertial>
-            <visual>
+<!--             <visual>
                 <geometry>
                     <mesh filename="package://hsrb_description/meshes/base_v2/bumper.dae"/>
@@ -222,5 +222,5 @@
                     <mesh filename="package://hsrb_description/meshes/base_v2/bumper.stl"/>
                 </geometry>
-            </collision>
+            </collision> -->
         </link>
         <joint name="${prefix}_roll_joint" type="continuous">

Commit message: made revolute hsr joints without axis and limits fixed

File: urdf/base_v2/base.urdf.xacro (robot description, xacro)
@@ -105,9 +105,8 @@
     <!-- bumper -->
     <xacro:macro name="hsrb_bumper" params="prefix suffix parent *origin">
-        <joint name="${prefix}_${suffix}_bumper_joint" type="revolute">
+        <joint name="${prefix}_${suffix}_bumper_joint" type="fixed">
             <xacro:insert_block name="origin" />
             <parent link="${parent}" />
             <child link="${prefix}_${suffix}_bumper_link" />
-            <limit effort="0" velocity="0" lower="0" upper="0"/>
         </joint>
         <link name="${prefix}_${suffix}_bumper_link">

File: urdf/sensors/minebea_ft_sensor.urdf.xacro (robot description, xacro)
@@ -3,9 +3,8 @@
     <xacro:include filename="$(find hsr_description)/urdf/sensors/minebea_ft_sensor.gazebo.xacro"/>
     <xacro:macro name="minebea_ft_sensor" params="prefix robot_namespace parent *origin">
-        <joint name="${prefix}_ft_sensor_frame_joint" type="revolute">
+        <joint name="${prefix}_ft_sensor_frame_joint" type="fixed">
             <xacro:insert_block name="origin"/>
             <parent link="${parent}"/>
             <child link="${prefix}_ft_sensor_frame"/>
-            <limit effort="100.0" velocity="1.5" lower="0" upper="0" />
         </joint>
         <link name="${prefix}_ft_sensor_frame">
